File: high-side-current-sense/kicad-src/high-side-current-sense.sch (KiCad schematic (older format))
At the start: 10 parts, among them J1 Conn_01x04, J2 Conn_01x04, U1 MAX4209HAUA

Commit message: stabilizes output with cap on FB pin
Parts:
- added C3: 10nF, Capacitor_SMD:C_0603_1608Metric, symbol Device:C_Small
Connections:
- wire segments 37 -> 39
Other:
- moved on the sheet: C2, R2
Changed lines of the file:
@@
 NoConn ~ 5450 3975
 Wire Wire Line
-	5450 3875 5375 3875
-Wire Wire Line
-	5375 3875 5375 4125
-Wire Wire Line
-	5375 4125 5750 4125
-Wire Wire Line
-	5450 3575 4700 3575
-Wire Wire Line
-	4700 3575 4700 4275
-Wire Wire Line
-	5000 4275 5000 3675
-Wire Wire Line
-	5000 3675 5450 3675
+	5450 3675 4700 3675
+Wire Wire Line
+	4700 3675 4700 4275
+Wire Wire Line
+	5000 4275 5000 3875
 $Comp
 L power:GND #PWR07
@@
 $EndComp
 Wire Wire Line
-	6625 3775 6950 3775
+	6825 3775 6950 3775
 $Comp
 L power:GND #PWR06
@@
 L Device:C_Small C2
 U 1 1 61AF9C54
-P 6350 3925
-F 0 "C2" H 6442 3971 50  0000 L CNN
-F 1 "1uF" H 6442 3880 50  0000 L CNN
-F 2 "Capacitor_SMD:C_0603_1608Metric" H 6350 3925 50  0001 C CNN
-F 3 "~" H 6350 3925 50  0001 C CNN
-	1    6350 3925
+P 6500 3925
+F 0 "C2" H 6592 3971 50  0000 L CNN
+F 1 "1uF" H 6592 3880 50  0000 L CNN
+F 2 "Capacitor_SMD:C_0603_1608Metric" H 6500 3925 50  0001 C CNN
+F 3 "~" H 6500 3925 50  0001 C CNN
+	1    6500 3925
 	1    0    0    -1
 $EndComp
@@
 L Device:R_Small R2
 U 1 1 61AFAEA8
-P 6525 3775
-F 0 "R2" V 6329 3775 50  0000 C CNN
-F 1 "100R" V 6420 3775 50  0000 C CNN
-F 2 "Resistor_SMD:R_0603_1608Metric" H 6525 3775 50  0001 C CNN
-F 3 "~" H 6525 3775 50  0001 C CNN
-	1    6525 3775
+P 6725 3775
+F 0 "R2" V 6529 3775 50  0000 C CNN
+F 1 "100R" V 6620 3775 50  0000 C CNN
+F 2 "Resistor_SMD:R_0603_1608Metric" H 6725 3775 50  0001 C CNN
+F 3 "~" H 6725 3775 50  0001 C CNN
+	1    6725 3775
 	0    1    1    0
 $EndComp
 Wire Wire Line
-	6350 4025 6350 4125
+	6500 4025 6500 4125
 Wire Wire Line
 	5750 4125 5850 4125
 Connection ~ 5850 4125
 Wire Wire Line
-	5850 4125 6350 4125
+	5850 4125 6500 4125
 Text Label 5075 4925 0    50   ~ 0
 SUPPLY+
@@
 	4675 4825 5400 4825
 Wire Wire Line
-	6250 3775 6350 3775
-Wire Wire Line
-	6350 3775 6350 3825
-Connection ~ 6350 3775
-Wire Wire Line
-	6350 3775 6425 3775
+	6500 3775 6500 3825
+Wire Wire Line
+	6500 3775 6625 3775
 $Comp
 L Mechanical:MountingHole H1
@@
 	1    0    0    -1
 $EndComp
+Wire Wire Line
+	5450 3875 5000 3875
+$Comp
+L Device:C_Small C3
+U 1 1 61A9D282
+P 6325 3925
+F 0 "C3" H 6400 3875 50  0000 L CNN
+F 1 "10nF" H 6400 3950 50  0000 L CNN
+F 2 "Capacitor_SMD:C_0603_1608Metric" H 6325 3925 50  0001 C CNN
+F 3 "~" H 6325 3925 50  0001 C CNN
+	1    6325 3925
+	-1   0    0    1
+$EndComp
+Wire Wire Line
+	6500 3775 6325 3775
+Connection ~ 6500 3775
+Wire Wire Line
+	6325 3775 6325 3825
+Connection ~ 6325 3775
+Wire Wire Line
+	6325 3775 6250 3775
+Wire Wire Line
+	5950 3975 5950 4075
+Wire Wire Line
+	5950 4075 6325 4075
+Wire Wire Line
+	6325 4075 6325 4025
 $EndSCHEMATC
