File: op-amp-low-side-current-sense/kicad-src/op-amp-low-side-current-sense.kicad_pcb (KiCad board)
At the start: 2 copper layers, 32.9 x 26.7 mm, 10 parts, among them J2 Conn_01x04, Q1 2N3904BU, U1 AD8551RM

Commit message: fix silkscreen error
Parts:
- renumbered C4 to C1
