File: non-contact-voltage-sensor/kicad-src/non-contact-voltage-sensor.sch (KiCad schematic (older format))
At the start: 19 parts, among them J1 Conn_01x05, Q1 BC547BTA, Q2 BC547BTA, Q3 BC547BTA, Q4 BC547BTA, Q5 BC557BTA, SW1 SW_SPST

Commit message: update render and prod files for diode
Parts:
- SW1: footprint (none) -> Button_Switch_SMD:SW_Push_1P1T_NO_6x6mm_H9.5mm
Changed lines of the file:
@@
 F 0 "SW1" H 7900 2685 50  0000 C CNN
 F 1 "SW_SPST" H 7900 2594 50  0000 C CNN
-F 2 "" H 7900 2450 50  0001 C CNN
+F 2 "Button_Switch_SMD:SW_Push_1P1T_NO_6x6mm_H9.5mm" H 7900 2450 50  0001 C CNN
 F 3 "~" H 7900 2450 50  0001 C CNN
 	1    7900 2450
