File: non-contact-voltage-sensor/kicad-src/non-contact-voltage-sensor.kicad_pcb (KiCad board)
At the start: 2 copper layers, 32.9 x 26.7 mm, 17 parts, among them J1 Conn_01x05, Q1 BC547BTA, Q2 BC547BTA, Q3 BC547BTA, Q4 BC547BTA, Q5 BC557BTA, SW1 SW_SPST

Commit message: update silkscreen for prod files
Other:
- board text added: "12/9/2021"
- board text removed: "12/13/2021"

Commit message: updates prod nc volt sensor
Other:
- board text added: "HV!"
