File: pwm-variable-motor-driver/kicad-src/pwm-variable-motor-driver.kicad_pcb (KiCad board)
At the start: 2 copper layers, 32.9 x 26.7 mm, 15 parts, among them J1 Conn_01x02, J2 Conn_01x02, Q1 AO3401A, U1 NE555DR

Commit message: minor change to pwm vr 3d model
Other:
- board text added: "12/11/2021"
- board text removed: "12/X/2021"
