File: boosted-output-current-reference/kicad-src/boosted-output-current-reference.kicad_pcb (KiCad board)
At the start: 2 copper layers, 32.9 x 26.7 mm, 15 parts, among them J1 Conn_01x02, J2 Conn_01x02, Q1 2N7002, U1 ADR425ARMZ, U2 AD8603

Commit message: add trim to v reference
Parts:
- added R2: 470K, Resistor_SMD:R_0603_1608Metric, F.Cu at (156.4, 99.0)
- added R3: 10K, Resistor_SMD:R_0603_1608Metric, F.Cu at (156.4, 103.2)
- added TRIM: 10K, Potentiometer_THT:Potentiometer_Bourns_3266W_Vertical, F.Cu at (153.8, 103.6)
- U1: value ADR425ARMZ -> ADR420BRZ
- renumbered TP1 to 2.048V
Routing:
- net Net-(R2-Pad2): track 0.00 -> 5.69 mm
- net Net-(C3-Pad2): track 8.69 -> 13.2 mm
- net Net-(R3-Pad1): track 0.00 -> 2.75 mm
- net Net-(R2-Pad1): track 0.00 -> 1.69 mm
- net GND: track 8.33 -> 9.37 mm, vias 15 -> 16
