File: portable-voltage-regulator/kicad-src/portable-voltage-regulator.kicad_pcb (KiCad board)
At the start: 2 copper layers, 30.7 x 26.7 mm, 13 parts, among them J1 Conn_01x03, Q1 IRF9540N, U1 ADR293GRUZ, U2 OPA333xxD

Commit message: upgrade opamp
Parts:
- U2: value OPA333xxD -> OPA188xxD
